Commit message: feat:add some test file and modify dir

File: model/franka_panda_urdf/robots/panda_arm.urdf (robot description, URDF)
Before this commit: robot panda, 9 links, 8 joints
Links:
- removed link panda_link0
- removed link panda_link1
- removed link panda_link2
- removed link panda_link3
- removed link panda_link4
- removed link panda_link5
- removed link panda_link6
- removed link panda_link7
- removed link panda_link8
- added link ee_center_body, mass 0.0
- added link hand, mass 0.0
- added link link0; collision mesh filename=meshes/collision/link0.stl; visual mesh filename=meshes/visual/link0.dae
- added link link1, mass 4.970684; collision mesh filename=meshes/collision/link1.stl; visual mesh filename=meshes/visual/link1.dae
- added link link2, mass 0.646926; collision mesh filename=meshes/collision/link2.stl; visual mesh filename=meshes/visual/link2.dae
- added link link3, mass 3.228604; collision mesh filename=meshes/collision/link3.stl; visual mesh filename=meshes/visual/link3.dae
- added link link4, mass 3.587895; collision mesh filename=meshes/collision/link4.stl; visual mesh filename=meshes/visual/link4.dae
- added link link5, mass 1.225946; collision mesh filename=meshes/collision/link5.stl; visual mesh filename=meshes/visual/link5.dae
- added link link6, mass 1.666555; collision mesh filename=meshes/collision/link6.stl; visual mesh filename=meshes/visual/link6.dae
- added link link7, mass 7.35522e-01; collision mesh filename=meshes/collision/link7.stl; visual mesh filename=meshes/visual/link7.dae
Joints:
- removed joint panda_joint1
- removed joint panda_joint2
- removed joint panda_joint3
- removed joint panda_joint4
- removed joint panda_joint5
- removed joint panda_joint6
- removed joint panda_joint7
- removed joint panda_joint8
- added joint joint1: type revolute, parent link0, child link1, origin xyz=0 0 0.333 rpy=0 0 0, axis 0 0 1, limit lower=-2.8973 upper=2.8973 effort=87 velocity=2.1750
- added joint joint2: type revolute, parent link1, child link2, origin xyz=0 0 0 rpy=-1.57079632679 0 0, axis 0 0 1, limit lower=-1.7628 upper=1.7628 effort=87 velocity=2.1750
- added joint joint3: type revolute, parent link2, child link3, origin xyz=0 -0.316 0 rpy=1.57079632679 0 0, axis 0 0 1, limit lower=-2.8973 upper=2.8973 effort=87 velocity=2.1750
- added joint joint4: type revolute, parent link3, child link4, origin xyz=0.0825 0 0 rpy=1.57079632679 0 0, axis 0 0 1, limit lower=-3.0718 upper=-0.0698 effort=87 velocity=2.1750
- added joint joint5: type revolute, parent link4, child link5, origin xyz=-0.0825 0.384 0 rpy=-1.57079632679 0 0, axis 0 0 1, limit lower=-2.8973 upper=2.8973 effort=12 velocity=2.6100
- added joint joint6: type revolute, parent link5, child link6, origin xyz=0 0 0 rpy=1.57079632679 0 0, axis 0 0 1, limit lower=-0.0175 upper=3.7525 effort=12 velocity=2.6100
- added joint joint7: type revolute, parent link6, child link7, origin xyz=0.088 0 0 rpy=1.57079632679 0 0, axis 0 0 1, limit lower=-2.8973 upper=2.8973 effort=12 velocity=2.6100
- added joint joint8: type fixed, parent link7, child hand, origin xyz=0 0 0.107 rpy=0 0 0, axis 0 0 0
- added joint joint9: type fixed, parent hand, child ee_center_body, origin xyz=0 0 0.105 rpy=0 0 0, axis 0 0 0
